File: Foinse.kicad_sch (KiCad schematic)
At the start: 54 parts, among them J1 Conn_ARM_JTAG_SWD_10, J2 2060-1452/998-404, J3 ESQ-110-14-G-D, J4 2060-1452/998-404, J5 2060-1452/998-404, J6 2060-1452/998-404, J7 2060-1452/998-404, J8 2601-1108, Q1 AO3400A, U1 STM32F072C8Tx, U2 TLV70433DBVT, U3 LTV-817, U4 TJA1051T-3, U5 TPS563203, U6 TPS563203

Commit message: Added E-Match circuit
Parts:
- added C30: 1 uF, symbol Device:C
- added D1: RED LED, symbol Device:LED
- added D2: GREEN LED, symbol Device:LED
- added Q2, Q3: AO3400A, Package_TO_SOT_SMD:SOT-23, symbol Transistor_FET:AO3400A
- added R10: 2 Ω, symbol Device:R
- added R11: 4.7 Ω, symbol Device:R
- added R12, R6: 10k Ω, symbol Device:R
- added R13: 1k Ω, symbol Device:R
- added R5: 220 Ω, symbol Device:R
- added R7: 1-3Ω, symbol Device:R
- added R8: 4.7k Ω, symbol Device:R
- added R9: 6 Ω, symbol Device:R
- added U7: LTV-817, Package_DIP:DIP-4_W7.62mm, symbol Isolator:LTV-817
Connections:
- net 3.3V: now also U7.4
- net GND: now also U3.2, R12.1
- net PGND: now also Q1.2 (S), Q2.2 (S), Q3.2 (S), R10.1, R6.2
- net VBAT_DROGUE: now also J8.1 (1_1), J8.2 (1_2), U3.4, C30.1, D1.1 (K), D2.1 (K), U7.1
- net at Q1.1 (G): now also U3.3, Q2.1 (G), R6.1
- net at Q1.3 (D): now also R7.1
- net Aux1 pos: now reaches J8.10 (5_2)
- net Aux1 pos: now also J8.9 (5_1)
- net Aux1 neg: now reaches J8.11 (6_1)
- net Aux1 neg: now also J8.12 (6_2)
- net Aux2 pos: now reaches J8.13 (7_1)
- net Aux2 pos: now also J8.14 (7_2)
- net Aux2 neg: now reaches J8.15 (8_1)
- net Aux2 neg: now also J8.16 (8_2)
- net Drogue neg: now reaches J8.3 (2_1)
- net Drogue neg: now also J8.4 (2_2), C30.2, R7.2, R9.2
- net Main pos: now reaches J8.5 (3_1)
- net Main pos: now also J8.6 (3_2)
- net Main neg: now reaches J8.7 (4_1)
- net Main neg: now also J8.8 (4_2)
- net at U3.1: now also R5.2
- net DROGUE_SEAT: now reaches U1.21 (PB10)
- net DROGUE_SEAT: now also R12.2, U7.3
- net MAIN_SEAT: now reaches U1.22 (PB11)
- net AUX1_SEAT: now reaches U1.25 (PB12)
- net AUX2_SEAT: now reaches U1.26 (PB13)
- net DROGUE_FIRE: now reaches U1.39 (PB3)
- net DROGUE_FIRE: now also R5.1
- net MAIN_FIRE: now reaches U1.40 (PB4)
- net AUX1_FIRE: now reaches U1.41 (PB5)
- net AUX2_FIRE: now reaches U1.42 (PB6)
- new net: R13.1, U7.2
- new net: Q3.1 (G), R10.2, R9.1
- new net: Q3.3 (D), R11.1, R13.2
- new net: Q2.3 (D), R8.1
- new net: D1.2 (A), R8.2
- new net: D2.2 (A), R11.2
Other:
- moved on the sheet: J1, J2, Q1, U3
