File: Foinse.kicad_sch (KiCad schematic)
At the start: 69 parts, among them J1 Conn_ARM_JTAG_SWD_10, J2 2060-1452/998-404, J3 ESQ-110-14-G-D, J4 2060-1452/998-404, J5 2060-1452/998-404, J6 2060-1452/998-404, J7 2060-1452/998-404, J8 2601-1108, Q1 AO3400A, Q2 AO3400A, Q3 AO3400A, U1 STM32F072C8Tx, U2 TLV70433DBVT, U3 LTV-817, U4 TJA1051T-3, U5 TPS563203, U6 TPS563203, U7 LTV-817

Commit message: Added E-Match circuit
Parts:
- added C31, C32, C33: 1 uF, symbol Device:C
- added D3, D5, D7: RED LED, symbol Device:LED
- added D4, D6, D8: GREEN LED, symbol Device:LED
- added Q10, Q11, Q12, Q4, Q5, Q6, Q7, Q8, Q9: AO3400A, Package_TO_SOT_SMD:SOT-23, symbol Transistor_FET:AO3400A
- added R14, R16, R23, R25, R32, R34: 10k Ω, symbol Device:R
- added R15, R24, R33: 220 Ω, symbol Device:R
- added R17, R26, R35: 1-3Ω, symbol Device:R
- added R18, R27, R36: 4.7k Ω, symbol Device:R
- added R19, R28, R37: 1k Ω, symbol Device:R
- added R20, R29, R38: 6 Ω, symbol Device:R
- added R21, R30, R39: 2 Ω, symbol Device:R
- added R22, R31, R40: 4.7 Ω, symbol Device:R
- added U10, U11, U12, U13, U8, U9: LTV-817, Package_DIP:DIP-4_W7.62mm, symbol Isolator:LTV-817
Connections:
- net Aux1 pos is gone; now on net VBAT_AUX1: J8.10 (5_2), J8.9 (5_1)
- net Aux2 pos is gone; now on net VBAT_AUX2: J8.13 (7_1), J8.14 (7_2)
- net Main pos is gone; now on net VBAT_MAIN: J8.5 (3_1), J8.6 (3_2)
- net 3.3V: now also U11.4, U13.4, U9.4
- net AUX1_FIRE: now also R24.1
- net AUX1_SEAT: now also R23.2, U11.3
- net AUX2_FIRE: now also R33.1
- net AUX2_SEAT: now also R32.2, U13.3
- net Aux1 neg: now also C32.2, R26.2, R29.2
- net Aux2 neg: now also C33.2, R35.2, R38.2
- net GND: now also R14.1, R23.1, R32.1, U10.2, U12.2, U8.2
- net MAIN_FIRE: now also R15.1
- net MAIN_SEAT: now also R14.2, U9.3
- net Main neg: now also C31.2, R17.2, R20.2
- net PGND: now also Q10.2 (S), Q11.2 (S), Q12.2 (S), Q4.2 (S), Q5.2 (S), Q6.2 (S), Q7.2 (S), Q8.2 (S), Q9.2 (S), R16.2, R21.1, R25.2, R30.1, R34.2, R39.1
- net VBAT_AUX1: now also C32.1, D5.2 (A), D6.2 (A), U10.4, U11.1
- net VBAT_AUX2: now also C33.1, D7.2 (A), D8.2 (A), U12.4, U13.1
- net VBAT_DROGUE: now also D1.2 (A), D2.2 (A); no longer D1.1 (K), D2.1 (K)
- net VBAT_MAIN: now also C31.1, D3.2 (A), D4.2 (A), U8.4, U9.1
- net at Q1.1 (G), Q2.1 (G), R6.1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: now also Q1.3 (D), R7.1
- net at R8.2: now also D1.1 (K); no longer D1.2 (A)
- net at R11.2: now also D2.1 (K); no longer D2.2 (A)
- new net: Q10.1 (G), Q10.3 (D), Q11.1 (G), R34.1, R35.1, U12.3
- new net: Q11.3 (D), R36.1
- new net: Q9.1 (G), R29.1, R30.2
- new net: Q9.3 (D), R28.2, R31.1
- new net: R15.2, U8.1
- new net: Q12.3 (D), R37.2, R40.1
- new net: D8.1 (K), R40.2
- new net: R33.2, U12.1
- new net: R19.1, U9.2
- new net: D6.1 (K), R31.2
- new net: D7.1 (K), R36.2
- new net: Q12.1 (G), R38.1, R39.2
- new net: R37.1, U13.2
- new net: D3.1 (K), R18.2
- new net: Q6.1 (G), R20.1, R21.2
- new net: Q4.1 (G), Q4.3 (D), Q5.1 (G), R16.1, R17.1, U8.3
- new net: D5.1 (K), R27.2
- new net: R28.1, U11.2
- new net: Q8.3 (D), R27.1
- new net: Q7.1 (G), Q7.3 (D), Q8.1 (G), R25.1, R26.1, U10.3
- new net: Q6.3 (D), R19.2, R22.1
- new net: D4.1 (K), R22.2
- new net: Q5.3 (D), R18.1
- new net: R24.2, U10.1
Other:
- note added: "E-Match Trigger Circuit"
- moved on the sheet: C1, C10, C11, C12, C13, C14, C15, C16, C17, C18, C19, C2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

Commit message: Board V1, before review
Parts:
- removed C23: 10 uF, symbol Device:C
- removed C24, C25, C29: 100 nF, symbol Device:C
- removed C26: 18 pF, symbol Device:C
- removed C27, C28: 22 uF, symbol Device:C
- removed J4, J6, J7: 2060-1452/998-404, footprints:WAG, symbol Wago_2060-1452 998-404:2060-1452_998-404
- removed L2: 4.7 uH, symbol Device:L
- removed R4: 100k Ω, symbol Device:R
- removed Ra1: 220 Ω, symbol Device:R
- removed Rb1: 30 Ω, symbol Device:R
- removed U6: TPS563203, Package_TO_SOT_SMD:SOT-563, symbol Regulator_Switching:TPS563203
- added C34, C35: 100nF, Capacitor_SMD:C_0402_1005Metric, symbol Device:C
- added C36: 47 nF, Capacitor_SMD:C_0402_1005Metric, symbol Device:C
- added C37, C40: 0.1 uF, Capacitor_SMD:C_0402_1005Metric, symbol Device:C
- added C38, C39: 10 uF, Capacitor_SMD:C_0402_1005Metric, symbol Device:C
- added C41: 150 pF, Capacitor_SMD:C_0402_1005Metric, symbol Device:C
- added C42, C43, C44, C45, C46: 22 uF, Capacitor_SMD:C_0402_1005Metric, symbol Device:C
- added D10: BAT54C, Package_TO_SOT_SMD:SOT-23, symbol Diode:BAT54C
- added D11, D12: RED LED, LED_SMD:LED_0402_1005Metric, symbol Device:LED
- added D14: D_Schottky, symbol Device:D_Schottky
- added D9: NUP2105L, Package_TO_SOT_SMD:SOT-23, symbol Power_Protection:NUP2105L
- added J10: Conn_02x03_Odd_Even, Connector_PinHeader_1.00mm:PinHeader_2x03_P1.00mm_Vertical, symbol Connector_Generic:Conn_02x03_Odd_Even
- added J4: PJ-002AH, Foinse Footprints:PJ-002AH_CUD, symbol PJ-002AH:PJ-002AH
- added J9: USB_C_Receptacle_USB2.0_16P, Connector_USB:USB_C_Receptacle_G-Switch_GT-USB-7010ASV, symbol Connector:USB_C_Receptacle_USB2.0_16P
- added L3: L_Iron, symbol Device:L_Iron
- added MOSFET1: IPP80P03P4L04AKSA1, Foinse Footprints:IPP80P03P4L04AKSA1, symbol IPP80P03P4L04AKSA1:IPP80P03P4L04AKSA1
- added Q13, Q14: AO3400A, Package_TO_SOT_SMD:SOT-23, symbol Transistor_FET:AO3400A
- added R41, R42: 5.1K, Resistor_SMD:R_0402_1005Metric, symbol Device:R
- added R43, R44: 10K, Resistor_SMD:R_0402_1005Metric, symbol Device:R
- added R45, R46: 10 mΩ, Resistor_SMD:R_0402_1005Metric, symbol Device:R
- added R47: 220 Ω, Resistor_SMD:R_0402_1005Metric, symbol Device:R
- added R48, R58: 10k Ω, Resistor_SMD:R_0402_1005Metric, symbol Device:R
- added R49: 4.7k Ω, Resistor_SMD:R_0402_1005Metric, symbol Device:R
- added R50: 3.3k Ω, Resistor_SMD:R_0402_1005Metric, symbol Device:R
- added R51: 52.3k Ω, Resistor_SMD:R_0402_1005Metric, symbol Device:R
- added R52: 169k Ω, Resistor_SMD:R_0402_1005Metric, symbol Device:R
- added R53: 36.1k Ω, Resistor_SMD:R_0402_1005Metric, symbol Device:R
- added R54, R57: DNP, Resistor_SMD:R_0402_1005Metric, symbol Device:R
- added R55: 49.9 Ω, Resistor_SMD:R_0402_1005Metric, symbol Device:R
- added R56: 73.2 Ω, Resistor_SMD:R_0402_1005Metric, symbol Device:R
- added U14: USBLC6-2SC6, Package_TO_SOT_SMD:SOT-23-6, symbol Power_Protection:USBLC6-2SC6
- added U15, U16: INA239AIDGSR, Foinse Footprints:VSSOP_9AIDGST_TEX, symbol INA239:INA239AIDGSR
- added U17: LTC4412xS6, Package_TO_SOT_SMD:TSOT-23-6, symbol Power_Management:LTC4412xS6
- added U18: LTV-817, Package_DIP:DIP-4_W7.62mm, symbol Isolator:LTV-817
- added U19: TPS56A37RPAR, Foinse Footprints:RPA0010A-MFG, symbol TPS56A37RPAR:TPS56A37RPAR
- C1, C10, C11, C12, C13, C14, C15, C16, C18, C19, C2, C20, C21, C22, C3, C30, C31, C32, C33, C4, C5, C6, C7, C8, C9: footprint (none) -> Capacitor_SMD:C_0402_1005Metric
- C17: value 100 nF -> 0.1 uF; footprint (none) -> Capacitor_SMD:C_0402_1005Metric
- D1, D2, D3, D4, D5, D6, D7, D8: footprint (none) -> LED_SMD:LED_0402_1005Metric
- J1: footprint (none) -> Connector_PinHeader_1.27mm:PinHeader_2x05_P1.27mm_Vertical
- J2: value 2060-1452/998-404 -> 2060-1452
- J3: footprint Connector_PinHeader_2.54mm:PinHeader_2x10_P2.54mm_Vertical -> Foinse Footprints:SAMTEC_ESQ-110-14-G-D
- J8: footprint Wago 2601-1104:CONN8_2601-1108_WAG -> Foinse Footprints:CONN8_2601-1108_WAG
- R1, R10, R11, R12, R13, R14, R15, R16, R17, R18, R19, R2, R20, R21, R22, R23, R24, R25, R26, R27, R28, R29, R3, R30, R31, R32, R33, R34, R35, R36, R37, R38, R39, R40, R5, R6, R7, R8, R9: footprint (none) -> Resistor_SMD:R_0402_1005Metric
- Ra2: renamed from Ra; footprint (none) -> Resistor_SMD:R_0402_1005Metric
- Rb2: renamed from Rb; footprint (none) -> Resistor_SMD:R_0402_1005Metric
Connections:
- net VBAT_AUX2 is gone; now on net VBAT_AUX1: C33.1, D7.2 (A), D8.2 (A), J8.13 (7_1), J8.14 (7_2), U12.4, U13.1
- net VBAT_DROGUE is gone; now on net VBAT_AUX1: C30.1, D1.2 (A), D2.2 (A), J2.1 (1_1), J2.2 (1_2), J8.1 (1_1), J8.2 (1_2), U3.4, U7.1
- net 3.3V: now also C34.1, C35.1, U15.6 (VS), U16.6 (VS)
- net 5VLOGIC: now also D10.2, R50.1; no longer C10.1, U2.2 (IN)
- net 5VSERVO: now also R46.2, U16.9 (IN-)
- net CAN_RX: no longer U1.32 (PA11)
- net CAN_TX: no longer U1.33 (PA12)
- net CAN_hi: no longer R2.1, U4.7 (CANH)
- net CAN_lo: no longer R1.2, U4.6 (CANL)
- net GND: now also J5.3 (2_1), J5.4 (2_2), C34.2, C35.2, C36.2, C37.2, C38.2, C39.2, D9.3 (A), J4.2, J9.A1 (GND), J9.A12 (GND), J9.B1 (GND), J9.B12 (GND), J9.S1 (SHIELD), R41.2, R42.1, R44.1, R51.2, R53.2, R58.2, U14.2 (GND), U15.7 (GND), U16.7 (GND), U17.2 (GND), U17.3 (CTL), U19.3 (AGND); no longer C16.1, C17.1, R12.1, R14.1, R23.1, R3.1, R32.1, U10.2, U12.2, U3.2, U5.1 (VIN), U8.2
- net PGND: now also R12.1, R14.1, R23.1, R32.1, U10.2, U12.2, U3.2, U8.2, Q14.3 (D), U18.2; no longer J2.3 (2_1), J2.4 (2_2), J5.3 (2_1), J5.4 (2_2)
- net SWCLK: now also U1.37 (PA14); no longer U1.3 (PC14)
- net SWDIO: now also U1.34 (PA13); no longer U1.2 (PC13)
- net VBAT_AUX1: now also C31.1, D3.2 (A), D4.2 (A), J8.5 (3_1), J8.6 (3_2), U8.4, U9.1, D11.2 (A), U18.4
- net SPI_CLK: now reaches U1.15 (PA5)
- net SPI_CLK: now also U15.5 (SCLK), U16.5 (SCLK)
- net SPI_MISO: now reaches U1.16 (PA6)
- net SPI_MISO: now also U15.4 (MISO), U16.4 (MISO)
- net SPI_MOSI: now reaches U1.17 (PA7)
- net SPI_MOSI: now also U15.2 (MOSI), U16.2 (MOSI)
- net BATTERY_CURRENT_CS: now reaches U1.27 (PB14)
- net BATTERY_CURRENT_CS: now also U15.1 (CS)
- net SERVO_CURRENT_CS: now reaches U1.28 (PB15)
- net SERVO_CURRENT_CS: now also U16.1 (CS)
- net PYRO_ON: now reaches U1.43 (PB7)
- net PYRO_ON: now also R47.1
- net Mode_sel: now reaches U1.45 (PB8)
- net Mode_sel: now also R43.1, R44.2
- removed net VBAT_MAIN: C31.1, D3.2 (A), D4.2 (A), J5.1 (1_1), J5.2 (1_2), J8.5 (3_1), J8.6 (3_2), U8.4, U9.1
- new net: C10.1, D10.3, U2.2 (IN)
- new net: R52.2, R53.1, U19.1 (EN)
- new net: D11.1 (K), Q13.1 (G), Q14.1 (G), R48.1, R49.2, U18.3
- new net: J2.3 (2_1), J2.4 (2_2), Q13.3 (D), Q14.2 (S), R48.2
- new net: D12.2 (A), R50.2
- new net: R47.2, U18.1
- new net: R55.2, R56.1, R57.2
- new net: C41.2, R56.2, R58.1, U19.2 (FB)
- new net: C40.2, L3.1, U19.6 (SW)
- new net: R54.1, U19.7 (BOOT)
- new net: C40.1, R54.2
- new net: J9.A7 (D-), J9.B7 (D-), U14.4 (I/O2)
- new net: J9.A6 (D+), J9.B6 (D+), U14.6 (I/O1)
- new net: J9.A5 (CC1), R41.1
- new net: C41.1, R57.1
- new net: MOSFET1.1 (G), U17.5 (GATE)
- new net: J5.1 (1_1), J5.2 (1_2), MOSFET1.2 (D), U17.1 (VIN)
- new net: C36.1, U19.5 (SS)
- new net: R51.1, U19.10 (MODE)
- new net: D14.2 (A), J4.1
- new net: D12.1 (K), U17.4 (STAT)
- new net: J9.B5 (CC2), R42.2
- new net: Q13.2 (S), R49.1
- new net 5VSERVO_BS: C42.1, C43.1, C44.1, C45.1, C46.1, L3.2, R46.1, R55.1, U16.10 (IN+), U16.8 (VBUS)
- new net CAN_+: J10.2 (Pin_2)
- new net CAN_-: J10.1 (Pin_1)
- new net CAN_BUS+: D9.1 (K), R2.1, U4.7 (CANH)
- new net CAN_BUS+-: D9.2 (K), R1.2, U4.6 (CANL)
- new net PA_+: J10.4 (Pin_4), U1.33 (PA12)
- new net PA_-: J10.3 (Pin_3), U1.32 (PA11)
- new net PGND2: C42.2, C43.2, C44.2, C45.2, C46.2, U19.9 (PGND)
- new net USB_D+: J10.6 (Pin_6), U14.1 (I/O1)
- new net USB_D-: J10.5 (Pin_5), U14.3 (I/O2)
- new net VBAT: C16.1, C17.1, C37.1, C38.1, C39.1, R3.1, R45.2, R52.1, U15.9 (IN-), U19.8 (VIN), U5.1 (VIN)
- new net VBAT_BS: D14.1 (K), MOSFET1.3 (S), R45.1, U15.10 (IN+), U15.8 (VBUS), U17.6 (SENSE)
- new net VBUS_RAW: D10.1, J9.A4 (VBUS), J9.A9 (VBUS), J9.B4 (VBUS), J9.B9 (VBUS), R43.2, U14.5 (VBUS)
- no-connect marks 2 -> 7
Other:
- note added: "Board Connectors"
- note added: "Current Sensing"
- note added: "Pyro Connectors"
- note added: "USB-C"
- note added: "USB-C & mode select"
- note removed: "Connectors"
- note removed: "Wago for main battery connection"
- moved on the sheet: C1, C10, C11, C12, C13, C14, C15, C16, C17, C18, C19, C2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
