File: hardware/Foinse.kicad_sch (KiCad schematic)
At the start: 73 parts, among them J1 ESQ-110-X-X-D, J2 XT30PW-M, J4 PJ-002AH, J6 JTAG-10 PIN, U1 STM32F072C8Tx, U15 INA239AIDGSR, U16 INA239AIDGSR, U17 LTC4412xS6, U19 TPS56A37RPAR, U2 TLV70433DBVT, U4 TJA1051T-3, U5 TPS563203

Commit message: hehe
Parts:
- removed R54, R57: 0, Resistor_SMD:R_0402_1005Metric, symbol Device:R
- added R6: 10k Ω, Resistor_SMD:R_0402_1005Metric, symbol Device:R
Connections:
- net 3.3V: now also R6.2
- net at R55.2, R56.1: now also C41.1
- net at U19.7 (BOOT): now also C40.1
- net at U19.4 (PG): now also R6.1
- no-connect marks 12 -> 11
Other:
- moved on the sheet: C40
Changed lines of the file:
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@@
 	)
 	(junction
+		(at 247.65 245.11)
+		(diameter 0)
+		(color 0 0 0 0)
+	)
+	(junction
 		(at 191.77 111.76)
 		(diameter 0)
@@
 	)
 	(junction
-		(at 247.65 246.38)
-		(diameter 0)
-		(color 0 0 0 0)
-	)
-	(junction
 		(at 194.31 318.77)
 		(diameter 0)
@@
 	)
 	(no_connect
-		(at 209.55 250.19)
-	)
-	(no_connect
 		(at 328.93 115.57)
 	)
@@
 	(wire
 		(pts
-			(xy 231.14 247.65) (xy 231.14 246.38)
+			(xy 231.14 247.65) (xy 231.14 245.11)
 		)
 		(stroke
@@
 	(wire
 		(pts
-			(xy 247.65 246.38) (xy 248.92 246.38)
-		)
-		(stroke
-			(width 0)
-			(type default)
-		)
-	)
-	(wire
-		(pts
 			(xy 411.8999 168.91) (xy 431.8 168.91)
 		)
@@
 	(wire
 		(pts
+			(xy 231.14 245.11) (xy 247.65 245.11)
+		)
+		(stroke
+			(width 0)
+			(type default)
+		)
+	)
+	(wire
+		(pts
 			(xy 209.55 308.61) (xy 222.25 308.61)
 		)
@@
 	(wire
 		(pts
-			(xy 209.55 237.49) (xy 210.82 237.49)
+			(xy 209.55 237.49) (xy 215.9 237.49)
 		)
 		(stroke
@@
 	(wire
 		(pts
-			(xy 247.65 246.38) (xy 247.65 247.65)
-		)
-		(stroke
-			(width 0)
-			(type default)
-		)
-	)
-	(wire
-		(pts
 			(xy 151.13 113.03) (xy 165.1 113.03)
 		)
@@
 	(wire
 		(pts
+			(xy 223.52 237.49) (xy 229.87 237.49)
+		)
+		(stroke
+			(width 0)
+			(type default)
+		)
+	)
+	(wire
+		(pts
 			(xy 285.75 160.02) (xy 285.75 154.94)
 		)
@@
 	(wire
 		(pts
-			(xy 231.14 246.38) (xy 236.22 246.38)
-		)
-		(stroke
-			(width 0)
-			(type default)
-		)
-	)
-	(wire
-		(pts
 			(xy 195.58 99.06) (xy 185.42 99.06)
 		)
@@
 	(wire
 		(pts
-			(xy 218.44 237.49) (xy 222.25 237.49)
-		)
-		(stroke
-			(width 0)
-			(type default)
-		)
-	)
-	(wire
-		(pts
 			(xy 336.55 330.2) (xy 342.9 330.2)
 		)
@@
 	(wire
 		(pts
-			(xy 243.84 246.38) (xy 247.65 246.38)
-		)
-		(stroke
-			(width 0)
-			(type default)
-		)
-	)
-	(wire
-		(pts
 			(xy 372.473 171.9473) (xy 385.173 171.9473)
 		)
@@
 	(wire
 		(pts
-			(xy 247.65 245.11) (xy 247.65 246.38)
+			(xy 247.65 245.11) (xy 247.65 247.65)
 		)
 		(stroke
@@
 		)
 	)
+	(global_label "3.3V"
+		(shape input)
+		(at 217.17 250.19 0)
+		(fields_autoplaced yes)
+		(effects
+			(font
+				(size 1.27 1.27)
+			)
+			(justify left)
+		)
+		(property "Intersheetrefs" "${INTERSHEET_REFS}"
+			(at 224.2676 250.19 0)
+			(effects
+				(font
+					(size 1.27 1.27)
+				)
+				(justify left)
+				(hide yes)
+			)
+		)
+	)
 	(symbol
 		(lib_id "power:GND")
@@
 	)
 	(symbol
-		(lib_id "Device:R")
-		(at 214.63 237.49 90)
-		(unit 1)
-		(exclude_from_sim no)
-		(in_bom yes)
-		(on_board yes)
-		(dnp no)
-		(property "Reference" "R54"
-			(at 214.63 239.776 90)
-			(effects
-				(font
-					(size 1.27 1.27)
-				)
-			)
-		)
-		(property "Value" "0"
-			(at 214.63 235.458 90)
-			(effects
-				(font
-					(size 1.27 1.27)
-				)
-			)
-		)
-		(property "Footprint" "Resistor_SMD:R_0402_1005Metric"
-			(at 214.63 239.268 90)
-			(effects
-				(font
-					(size 1.27 1.27)
-				)
-				(hide yes)
-			)
-		)
-		(property "Datasheet" "~"
-			(at 214.63 237.49 0)
-			(effects
-				(font
-					(size 1.27 1.27)
-				)
-				(hide yes)
-			)
-		)
-		(property "Description" "Resistor"
-			(at 214.63 237.49 0)
-			(effects
-				(font
-					(size 1.27 1.27)
-				)
-				(hide yes)
-			)
-		)
-		(pin "1"
-		)
-		(pin "2"
-		)
-		(instances
-			(project "Foinse"
-				(path "/e25e400c-9bc4-4e0b-8f6d-7db79788ea60"
-					(reference "R54")
-					(unit 1)
-				)
-			)
-		)
-	)
-	(symbol
 		(lib_id "power:GND")
 		(at 170.18 276.86 0)
@@
 	)
 	(symbol
-		(lib_id "Device:R")
-		(at 240.03 246.38 90)
-		(unit 1)
-		(exclude_from_sim no)
-		(in_bom yes)
-		(on_board yes)
-		(dnp no)
-		(property "Reference" "R57"
-			(at 240.03 248.666 90)
-			(effects
-				(font
-					(size 1.27 1.27)
-				)
-			)
-		)
-		(property "Value" "0"
-			(at 240.03 244.348 90)
-			(effects
-				(font
-					(size 1.27 1.27)
-				)
-			)
-		)
-		(property "Footprint" "Resistor_SMD:R_0402_1005Metric"
-			(at 240.03 248.158 90)
-			(effects
-				(font
-					(size 1.27 1.27)
-				)
-				(hide yes)
-			)
-		)
-		(property "Datasheet" "~"
-			(at 240.03 246.38 0)
-			(effects
-				(font
-					(size 1.27 1.27)
-				)
-				(hide yes)
-			)
-		)
-		(property "Description" "Resistor"
-			(at 240.03 246.38 0)
-			(effects
-				(font
-					(size 1.27 1.27)
-				)
-				(hide yes)
-			)
-		)
-		(pin "1"
-		)
-		(pin "2"
-		)
-		(instances
-			(project "Foinse"
-				(path "/e25e400c-9bc4-4e0b-8f6d-7db79788ea60"
-					(reference "R57")
-					(unit 1)
-				)
-			)
-		)
-	)
-	(symbol
 		(lib_id "power:GND")
 		(at 195.58 101.6 0)
@@
 	)
 	(symbol
+		(lib_id "Device:R")
+		(at 213.36 250.19 90)
+		(unit 1)
+		(exclude_from_sim no)
+		(in_bom yes)
+		(on_board yes)
+		(dnp no)
+		(property "Reference" "R6"
+			(at 213.36 252.476 90)
+			(effects
+				(font
+					(size 1.27 1.27)
+				)
+			)
+		)
+		(property "Value" "10k Ω"
+			(at 213.36 248.158 90)
+			(effects
+				(font
+					(size 1.27 1.27)
+				)
+			)
+		)
+		(property "Footprint" "Resistor_SMD:R_0402_1005Metric"
+			(at 213.36 251.968 90)
+			(effects
+				(font
+					(size 1.27 1.27)
+				)
+				(hide yes)
+			)
+		)
+		(property "Datasheet" "~"
+			(at 213.36 250.19 0)
+			(effects
+				(font
+					(size 1.27 1.27)
+				)
+				(hide yes)
+			)
+		)
+		(property "Description" "Resistor"
+			(at 213.36 250.19 0)
+			(effects
+				(font
+					(size 1.27 1.27)
+				)
+				(hide yes)
+			)
+		)
+		(pin "1"
+		)
+		(pin "2"
+		)
+		(instances
+			(project "Foinse"
+				(path "/e25e400c-9bc4-4e0b-8f6d-7db79788ea60"
+					(reference "R6")
+					(unit 1)
+				)
+			)
+		)
+	)
+	(symbol
 		(lib_id "Device:C")
 		(at 422.003 189.7273 90)
@@
 	(symbol
 		(lib_id "Device:C")
-		(at 226.06 237.49 90)
+		(at 219.71 237.49 90)
 		(unit 1)
 		(exclude_from_sim no)
@@
 		(dnp no)
 		(property "Reference" "C40"
-			(at 227.838 241.046 90)
+			(at 221.488 241.046 90)
 			(effects
 				(font
@@
 		)
 		(property "Value" "0.1 uF"
-			(at 228.854 234.188 90)
+			(at 222.504 234.188 90)
 			(effects
 				(font
@@
 		)
 		(property "Footprint" "Capacitor_SMD:C_0402_1005Metric"
-			(at 229.87 236.5248 0)
+			(at 223.52 236.5248 0)
 			(effects
 				(font
@@
 		)
 		(property "Datasheet" "~"
-			(at 226.06 237.49 0)
+			(at 219.71 237.49 0)
 			(effects
 				(font
@@
 		)
 		(property "Description" "Unpolarized capacitor"
-			(at 226.06 237.49 0)
+			(at 219.71 237.49 0)
 			(effects
 				(font

Commit message: hehe
Connections:
- net GND: now also J4.3
- no-connect marks 11 -> 10
Other:
- moved on the sheet: C41, R58
Changed lines of the file:
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@@
 	)
 	(junction
+		(at 307.34 191.77)
+		(diameter 0)
+		(color 0 0 0 0)
+	)
+	(junction
 		(at 146.05 237.49)
 		(diameter 0)
@@
 	)
 	(junction
+		(at 231.14 265.43)
+		(diameter 0)
+		(color 0 0 0 0)
+	)
+	(junction
 		(at 123.19 102.87)
 		(diameter 0)
@@
 	)
 	(no_connect
-		(at 307.34 194.31)
-	)
-	(no_connect
 		(at 328.93 115.57)
 	)
@@
 	(wire
 		(pts
+			(xy 307.34 191.77) (xy 307.34 194.31)
+		)
+		(stroke
+			(width 0)
+			(type default)
+		)
+	)
+	(wire
+		(pts
 			(xy 355.6 273.05) (xy 356.87 273.05)
 		)
@@
 	(wire
 		(pts
-			(xy 231.14 247.65) (xy 231.14 245.11)
+			(xy 231.14 246.38) (xy 231.14 245.11)
 		)
 		(stroke
@@
 	(wire
 		(pts
+			(xy 231.14 254) (xy 231.14 255.27)
+		)
+		(stroke
+			(width 0)
+			(type default)
+		)
+	)
+	(wire
+		(pts
 			(xy 212.09 102.87) (xy 201.93 102.87)
 		)
@@
 	(wire
 		(pts
-			(xy 231.14 265.43) (xy 231.14 264.16)
+			(xy 231.14 266.7) (xy 231.14 265.43)
 		)
 		(stroke
@@
 	(wire
 		(pts
-			(xy 231.14 255.27) (xy 231.14 256.54)
+			(xy 231.14 255.27) (xy 231.14 257.81)
 		)
 		(stroke
@@
 	(symbol
 		(lib_id "Device:R")
-		(at 231.14 260.35 0)
+		(at 231.14 261.62 0)
 		(unit 1)
 		(exclude_from_sim no)
@@
 		(dnp no)
 		(property "Reference" "R58"
-			(at 228.854 260.35 90)
+			(at 228.854 261.62 90)
 			(effects
 				(font
@@
 		)
 		(property "Value" "10k Ω"
-			(at 233.172 260.35 90)
+			(at 233.172 261.62 90)
 			(effects
 				(font
@@
 		)
 		(property "Footprint" "Resistor_SMD:R_0402_1005Metric"
-			(at 229.362 260.35 90)
+			(at 229.362 261.62 90)
 			(effects
 				(font
@@
 		)
 		(property "Datasheet" "~"
-			(at 231.14 260.35 0)
+			(at 231.14 261.62 0)
 			(effects
 				(font
@@
 		)
 		(property "Description" "Resistor"
-			(at 231.14 260.35 0)
+			(at 231.14 261.62 0)
 			(effects
 				(font
@@
 	(symbol
 		(lib_id "Device:C")
-		(at 231.14 251.46 0)
+		(at 231.14 250.19 0)
 		(unit 1)
 		(exclude_from_sim no)
@@
 		(dnp no)
 		(property "Reference" "C41"
-			(at 226.822 248.92 0)
+			(at 226.822 247.65 0)
 			(effects
 				(font
@@
 		)
 		(property "Value" "150 pF"
-			(at 231.394 253.746 0)
+			(at 231.394 252.476 0)
 			(effects
 				(font
@@
 		)
 		(property "Footprint" "Capacitor_SMD:C_0402_1005Metric"
-			(at 232.1052 255.27 0)
+			(at 232.1052 254 0)
 			(effects
 				(font
@@
 		)
 		(property "Datasheet" "~"
-			(at 231.14 251.46 0)
+			(at 231.14 250.19 0)
 			(effects
 				(font
@@
 		)
 		(property "Description" "Unpolarized capacitor"
-			(at 231.14 251.46 0)
+			(at 231.14 250.19 0)
 			(effects
 				(font

Commit message: never
Connections:
- net 5v_SERVO is gone; now on net 5VSERVO_BS: J1.01, J1.02
- net VBAT: now also D14.1 (K), MOSFET1.3 (S), U17.6 (SENSE)
- net VBAT_BS: no longer D14.1 (K), MOSFET1.3 (S), U17.6 (SENSE)
Changed lines of the file:
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@@
+		)
+	)
+	(label "???"
+		(at 276.86 154.94 0)
+		(effects
+			(font
+				(size 1.27 1.27)
+			)
+			(justify left bottom)
 		)
 	)
@@
 		)
 	)
-	(global_label "5v_SERVO"
+	(global_label "5VSERVO_BS"
 		(shape input)
 		(at 287.02 113.03 0)
@@
 		)
 		(property "Intersheetrefs" "${INTERSHEET_REFS}"
-			(at 299.1975 113.03 0)
+			(at 301.798 113.03 0)
 			(effects
 				(font
@@
 		)
 	)
-	(global_label "VBAT_BS"
+	(global_label "VBAT"
 		(shape input)
 		(at 304.8 162.56 180)
@@
 		)
 		(property "Intersheetrefs" "${INTERSHEET_REFS}"
-			(at 293.9529 162.56 0)
-			(effects
-				(font
+			(at 297.4 162.56 0)
+			(effects
+				(font
