File: hardware/power.kicad_sch (KiCad schematic)
At the start: 0 parts

Commit message: minor stuff
Parts:
- added C10: 39pf, Capacitor_SMD:C_0402_1005Metric, symbol Device:C
- added C11, C31: 0.1uf, Capacitor_SMD:C_0402_1005Metric, symbol Device:C
- added C29, C30, C34, C35, C47, C48: 22uf, Capacitor_SMD:C_0402_1005Metric, symbol Device:C
- added C33: 1uf, Capacitor_SMD:C_0402_1005Metric, symbol Device:C
- added C49, C50: 4.7uf, Capacitor_SMD:C_0402_1005Metric, symbol Device:C
- added C51: 10uf, Capacitor_SMD:C_0402_1005Metric, symbol Device:C
- added R10, R9: 0Ω, Resistor_SMD:R_0402_1005Metric, symbol Device:R
- added R11: 499kΩ, Resistor_SMD:R_0402_1005Metric, symbol Device:R
- added R12: 100kΩ, Resistor_SMD:R_0402_1005Metric, symbol Device:R
- added R13: 33.2kΩ, Resistor_SMD:R_0402_1005Metric, symbol Device:R
- added R4: 10kΩ, Resistor_SMD:R_0402_1005Metric, symbol Device:R
- added R8: 53.6kΩ, Resistor_SMD:R_0402_1005Metric, symbol Device:R
- added U2: MPM3650CGQW-P, QFN-24_MPM3650_MNP, symbol MPM3650CGQW-P:MPM3650CGQW-P
- added VR1: LT3045EDD_PBF, SON50P300X300X80-11N, symbol LT3045EDD_PBF:LT3045EDD_PBF
Connections:
- new net: C10.2, R4.2, R8.1, R9.1
- new net: R9.2, U2.17 (FB)
- new net: C10.1, C31.1, C34.1, C35.1, C47.1, C48.1, C50.2, R8.2, U2.10 (OUT), U2.11 (OUT), U2.12 (OUT), U2.9 (OUT), VR1.1 (IN_1), VR1.2 (IN_2), VR1.3 (EN/UV), VR1.6 (PGFB)
- new net: C49.2, R13.1, VR1.7 (SET)
- new net: R12.1, U2.20 (PG), U2.21 (PG)
- new net: C33.2, R12.2, U2.6 (VCC)
- new net: R11.1, U2.16 (EN)
- new net 3.3v: C51.1, VR1.10 (OUT), VR1.9 (OUTS)
- new net AGND: C33.1, R10.1, R4.1, U2.18 (AGND)
- new net GND: C11.1, C29.1, C30.1, C31.2, C34.2, C35.2, C47.2, C48.2, C49.1, C50.1, C51.2, R10.2, R13.2, U2.1 (PGND), U2.2 (PGND), U2.24 (PGND), U2.3 (PGND), U2.4 (PGND), U2.5 (PGND), VR1.11 (EXP), VR1.5 (ILIM), VR1.8 (GND)
- new net vin: C11.2, C29.2, C30.2, R11.2, U2.22 (VIN)
- no-connect marks 0 -> 8
Other:
- note added: "10kΩ"
- note added: "3.8v out"
- note added: "53.6kΩ"
- note added: "R2 = 10.0kΩ + R1 = 53.6kΩ"
- note added: "r1"
- note added: "r2"

Commit message: minor changes
Parts:
- removed C49: 4.7uf, Capacitor_SMD:C_0402_1005Metric, symbol Device:C
- removed R10, R9: 0Ω, Resistor_SMD:R_0402_1005Metric, symbol Device:R
- removed R11: 499kΩ, Resistor_SMD:R_0402_1005Metric, symbol Device:R
- removed R13: 33.2kΩ, Resistor_SMD:R_0402_1005Metric, symbol Device:R
- removed VR1: LT3045EDD_PBF, SON50P300X300X80-11N, symbol LT3045EDD_PBF:LT3045EDD_PBF
- added U8: TLV75533PDRV, Package_SON:WSON-6-1EP_2x2mm_P0.65mm_EP1x1.6mm, symbol Regulator_Linear:TLV75533PDRV
- C50: value 4.7uf -> 1uf
- C51: value 10uf -> 1uf
Connections:
- net AGND is gone; now on net GND: C33.1, R4.1, U2.18 (AGND)
- net 3.3v: now also U8.1 (OUT)
- net GND: now also U8.3 (GND), U8.7 (GND)
- net vin: now also U2.16 (EN)
- net at C10.2, R4.2, R8.1: now also U2.17 (FB)
- net at C10.1, C31.1, C34.1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: now also U8.4 (EN), U8.6 (IN)
- no-connect marks 8 -> 7
Other:
- note added: "what value should these caps be?"
- note removed: "10kΩ"
- note removed: "53.6kΩ"
- note removed: "r1"
- note removed: "r2"
- moved on the sheet: C11, C29, C30, C31, C34, C35, C47, C48, C50, C51, R12

Commit message: cleaned up component sizes
Parts:
- C29, C30, C34, C35, C47, C48: footprint Capacitor_SMD:C_0402_1005Metric -> Capacitor_SMD:C_0603_1608Metric
- U2: footprint QFN-24_MPM3650_MNP -> footprints:QFN-24_MPM3650_MNP
Changed lines of the file:
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@@
 			)
 		)
-		(property "Footprint" "Capacitor_SMD:C_0402_1005Metric"
+		(property "Footprint" "Capacitor_SMD:C_0603_1608Metric"
 			(at 52.3748 86.36 0)
 			(effects
@@
 			)
 		)
-		(property "Footprint" "Capacitor_SMD:C_0402_1005Metric"
+		(property "Footprint" "Capacitor_SMD:C_0603_1608Metric"
 			(at 115.2652 71.12 0)
 			(effects
@@
 			)
 		)
-		(property "Footprint" "Capacitor_SMD:C_0402_1005Metric"
+		(property "Footprint" "Capacitor_SMD:C_0603_1608Metric"
 			(at 127.9652 71.12 0)
 			(effects
@@
 			)
 		)
-		(property "Footprint" "Capacitor_SMD:C_0402_1005Metric"
+		(property "Footprint" "Capacitor_SMD:C_0603_1608Metric"
 			(at 134.3152 71.12 0)
 			(effects
@@
 			)
 		)
-		(property "Footprint" "QFN-24_MPM3650_MNP"
+		(property "Footprint" "footprints:QFN-24_MPM3650_MNP"
 			(at 105.41 91.44 0)
 			(effects
@@
 			)
 		)
-		(property "Footprint" "Capacitor_SMD:C_0402_1005Metric"
+		(property "Footprint" "Capacitor_SMD:C_0603_1608Metric"
 			(at 58.7248 86.36 0)
 			(effects
@@
 			)
 		)
-		(property "Footprint" "Capacitor_SMD:C_0402_1005Metric"
+		(property "Footprint" "Capacitor_SMD:C_0603_1608Metric"
 			(at 121.6152 71.12 0)
 			(effects
